Commit message: link to my gazebo ok

File: legacy/unitree_go2_description/xacro/robot.xacro (robot description, xacro)
@@ -69,10 +69,10 @@
         <collision>
             <origin rpy="0 0 0" xyz="0 0 0"/>
+            <!-- <geometry>
+                <mesh filename="file://$(find unitree_go2_description)/meshes/trunk.dae" scale="1 1 1"/>
+            </geometry> -->
             <geometry>
-                <mesh filename="file://$(find unitree_go2_description)/meshes/trunk.dae" scale="1 1 1"/>
+                <box size="${trunk_length} ${trunk_width} ${trunk_height}"/>
             </geometry>
-            <!-- <geometry>
-                <box size="${trunk_length} ${trunk_width} ${trunk_height}"/>
-            </geometry> -->
         </collision>
         <inertial>
