Commit message: r

File: legacy/unitree_go2_description/xacro/const.xacro (robot description, xacro)
@@ -1,11 +1,12 @@
 <?xml version="1.0"?>
 <robot xmlns:xacro="http://www.ros.org/wiki/xacro">
+    <!--总重：13.5，腿重：1.9，腿不含hip电机-->
     <!-- Constants for robot dimensions -->
     <xacro:property name="PI" value="3.1415926535897931"/>
     <xacro:property name="stick_mass" value="0.00001"/>
     <!-- simplified collision value -->
-    <xacro:property name="trunk_width" value="0.0935"/>
-    <xacro:property name="trunk_length" value="0.3762"/>
-    <xacro:property name="trunk_height" value="0.114"/>
+    <xacro:property name="trunk_width" value="0.25"/>
+    <xacro:property name="trunk_length" value="0.26"/>
+    <xacro:property name="trunk_height" value="0.12"/>
     <xacro:property name="hip_radius" value="0.046"/>
     <xacro:property name="hip_length" value="0.04"/>
@@ -16,23 +17,27 @@
     <xacro:property name="calf_width" value="0.016"/>
     <xacro:property name="calf_height" value="0.016"/>
-    <xacro:property name="foot_radius" value="0.02"/>
+    <xacro:property name="foot_radius" value="0.035"/>
     <xacro:property name="stick_radius" value="0.01"/>
     <xacro:property name="stick_length" value="0.2"/>
     <!-- kinematic value -->
-    <xacro:property name="thigh_offset" value="0.0955"/>
-    <xacro:property name="thigh_length" value="0.213"/>
-    <xacro:property name="calf_length" value="0.213"/>
+    <xacro:property name="thigh_offset" value="0.08"/>  <!--标识大腿板距离calf电机的偏移-->
+    <xacro:property name="thigh_length" value="0.15"/>  <!--标识大腿长度，以及calf电机的关节偏移-->
+    <xacro:property name="calf_length" value="0.15"/>
     <!-- leg offset from trunk center value -->
-    <xacro:property name="leg_offset_x" value="0.1934"/>
-    <xacro:property name="leg_offset_y" value="0.0465"/>
+    <!-- <xacro:property name="leg_offset_x" value="0.1934"/>
+    <xacro:property name="leg_offset_y" value="0.0465"/> -->
+    <xacro:property name="leg_offset_x" value="0.226"/>
+    <xacro:property name="leg_offset_y" value="0.085"/>
     <!-- <xacro:property name="trunk_offset_z" value="0.01675"/> -->
-    <xacro:property name="hip_offset" value="0.0955"/>
+    <xacro:property name="hip_offset" value="0.0955"/>  <!--标识了hip的碰撞偏移属性-->
     <!-- offset of link locations (left front) -->
     <xacro:property name="hip_offset_x" value="0.1934"/>
     <xacro:property name="hip_offset_y" value="0.0465"/>
     <xacro:property name="hip_offset_z" value="0.0"/>
+    <!--未使用参数-->
     <xacro:property name="thigh_offset_x" value="0"/>
     <xacro:property name="thigh_offset_y" value="0.0955"/>
     <xacro:property name="thigh_offset_z" value="0.0"/>
+    <!--未使用参数-->
     <xacro:property name="calf_offset_x" value="0.0"/>
     <xacro:property name="calf_offset_y" value="0.0"/>
@@ -45,19 +50,22 @@
     <xacro:property name="hip_velocity_max" value="30.1"/>
     <xacro:property name="hip_torque_max" value="23.7"/>
+    <!-- <xacro:property name="hip_torque_max" value="30"/> -->
     <xacro:property name="thigh_position_max" value="3.4907"/>
     <xacro:property name="thigh_position_min" value="-1.5708"/>
     <xacro:property name="thigh_velocity_max" value="30.1"/>
     <xacro:property name="thigh_torque_max" value="23.7"/>
+    <!-- <xacro:property name="thigh_torque_max" value="30"/> -->
     <xacro:property name="calf_position_max" value="-0.83776"/>
     <xacro:property name="calf_position_min" value="-2.7227"/>
     <xacro:property name="calf_velocity_max" value="20.06"/>
     <xacro:property name="calf_torque_max" value="35.55"/>
+    <!-- <xacro:property name="calf_torque_max" value="40"/> -->
     <!-- dynamics inertial value -->
     <!-- trunk -->
-    <xacro:property name="trunk_mass" value="6.921"/>
-    <xacro:property name="trunk_com_x" value="0.021112"/>
+    <xacro:property name="trunk_mass" value="5.9"/>       <!--躯干质量-->
+    <xacro:property name="trunk_com_x" value="0.021112"/>   <!--定义了惯性矩阵的质心（质心位置）相对于链接坐标系的偏移-->
     <xacro:property name="trunk_com_y" value="0.00"/>
     <xacro:property name="trunk_com_z" value="-0.005366"/>
-    <xacro:property name="trunk_ixx" value="0.02448"/>
+    <xacro:property name="trunk_ixx" value="0.02448"/>      <!--躯干的惯性矩阵 -->
     <xacro:property name="trunk_ixy" value="0.00012166"/>
     <xacro:property name="trunk_ixz" value="0.0014849"/>
@@ -65,6 +73,13 @@
     <xacro:property name="trunk_iyz" value="-3.12E-05"/>
     <xacro:property name="trunk_izz" value="0.107"/>
+    <!-- <xacro:property name="trunk_ixx" value="0.03780912"/>
+    <xacro:property name="trunk_ixy" value="0.0"/>
+    <xacro:property name="trunk_ixz" value="0.0"/>
+    <xacro:property name="trunk_iyy" value="0.0403167"/>
+    <xacro:property name="trunk_iyz" value="0"/>
+    <xacro:property name="trunk_izz" value="0.0639658"/> -->
     <!-- hip (left front) -->
-    <xacro:property name="hip_mass" value="0.678"/>
+    <!-- <xacro:property name="hip_mass" value="0.678"/> -->
+    <xacro:property name="hip_mass" value="0.91"/>
     <xacro:property name="hip_com_x" value="-0.0054"/>
     <xacro:property name="hip_com_y" value="0.00194"/>
@@ -77,5 +92,6 @@
     <xacro:property name="hip_izz" value="0.000596"/>
     <!-- thigh -->
-    <xacro:property name="thigh_mass" value="1.152"/>
+    <!-- <xacro:property name="thigh_mass" value="1.152"/> -->
+    <xacro:property name="thigh_mass" value="0.89"/>
     <xacro:property name="thigh_com_x" value="-0.00374"/>
     <xacro:property name="thigh_com_y" value="-0.0223"/>
@@ -88,5 +104,6 @@
     <xacro:property name="thigh_izz" value="0.00103"/>
     <!-- calf -->
-    <xacro:property name="calf_mass" value="0.154"/>
+    <!-- <xacro:property name="calf_mass" value="0.1"/> -->
+    <xacro:property name="calf_mass" value="0.1"/>
     <xacro:property name="calf_com_x" value="0.00548"/>
     <xacro:property name="calf_com_y" value="-0.000975"/>

File: legacy/unitree_go2_description/xacro/leg.xacro (robot description, xacro)
@@ -18,8 +18,8 @@
             <child link="${name}_hip"/>
             <axis xyz="1 0 0"/>
-            <dynamics damping="${damping}" friction="${friction}"/>
+            <dynamics damping="${damping}" friction="${friction}"/>   <!-- damping,friction对应gazebo中的阻尼系数和摩擦系数 -->
             <xacro:if value="${(mirror_dae == True)}">
                 <limit effort="${hip_torque_max}" velocity="${hip_velocity_max}" lower="${hip_position_min}"
-                       upper="${hip_position_max}"/>
+                       upper="${hip_position_max}"/>    <!--关节的力，速度，位置限幅-->
             </xacro:if>
             <xacro:if value="${(mirror_dae == False)}">
@@ -31,17 +31,18 @@
             <visual>
                 <xacro:if value="${(mirror_dae == True) and (front_hind_dae == True)}">
-                    <origin rpy="0 0 0" xyz="0 0 0"/>
+                    <origin rpy="0 ${PI} ${-PI/2.0}" xyz="0 0 0"/>
                 </xacro:if>
                 <xacro:if value="${(mirror_dae == False) and (front_hind_dae == True)}">
-                    <origin rpy="${PI} 0 0" xyz="0 0 0"/>
+                    <origin rpy="${PI} ${PI} ${PI/2.0}" xyz="0 0 0"/>
                 </xacro:if>
                 <xacro:if value="${(mirror_dae == True) and (front_hind_dae == False)}">
-                    <origin rpy="0 ${PI} 0" xyz="0 0 0"/>
+                    <origin rpy="${PI} ${PI} ${-PI/2.0}" xyz="0 0 0"/>
                 </xacro:if>
                 <xacro:if value="${(mirror_dae == False) and (front_hind_dae == False)}">
-                    <origin rpy="${PI} ${PI} 0" xyz="0 0 0"/>
+                    <origin rpy="0 ${PI} ${PI/2.0}" xyz="0 0 0"/>
                 </xacro:if>
                 <geometry>
-                    <mesh filename="file://$(find unitree_go2_description)/meshes/hip.dae" scale="1 1 1"/>
+                    <!-- <mesh filename="file://$(find unitree_go2_description)/meshes/hip.dae" scale="1 1 1"/> -->
+                    <mesh filename="package://unitree_go2_description/meshes/link1.STL" />
                 </geometry>
             </visual>
@@ -72,13 +73,25 @@
         <link name="${name}_thigh">
             <visual>
-                <origin rpy="0 0 0" xyz="0 0 0"/>
-                <geometry>
-                    <xacro:if value="${mirror_dae == True}">
-                        <mesh filename="file://$(find unitree_go2_description)/meshes/thigh.dae" scale="1 1 1"/>
+                <xacro:if value="${mirror_dae == True}">
+                    <origin rpy="0 0 ${PI/2.0}" xyz="0 0 0"/>
+                    <geometry>
+                        <mesh filename="package://unitree_go2_description/meshes/link2.STL" />
+                    </geometry>
+                </xacro:if>
+                <xacro:if value="${mirror_dae == False}">
+                    <origin rpy="0 0 ${-PI/2.0}" xyz="0 0 0"/>
+                    <geometry>
+                        <mesh filename="package://unitree_go2_description/meshes/link2.STL" />
+                    </geometry>
+                </xacro:if>
+                        <!-- <origin rpy="0 0 ${PI/2.0}" xyz="0 0 0"/> -->
+                        <!-- <mesh filename="file://$(find unitree_go2_description)/meshes/thigh.dae" scale="1 1 1"/> -->
+                        <!-- <mesh filename="package://unitree_go2_description/meshes/link2.STL" />
                     </xacro:if>
-                    <xacro:if value="${mirror_dae == False}">
-                        <mesh filename="file://$(find unitree_go2_description)/meshes/thigh_mirror.dae" scale="1 1 1"/>
-                    </xacro:if>
-                </geometry>
+                    <xacro:if value="${mirror_dae == False}"> -->
+                        <!-- <origin rpy="0 0 ${-PI/2.0}" xyz="0 0 0"/> -->
+                        <!-- <mesh filename="file://$(find unitree_go2_description)/meshes/thigh_mirror.dae" scale="1 1 1"/> -->
+                        <!-- <mesh filename="package://unitree_go2_description/meshes/link2.STL" />
+                    </xacro:if>  -->
             </visual>
             <collision>
@@ -108,7 +121,8 @@
         <link name="${name}_calf">
             <visual>
-                <origin rpy="0 0 0" xyz="0 0 0"/>
+                <origin rpy="0 0 ${PI/2.0}" xyz="0 0 0"/>
                 <geometry>
-                    <mesh filename="file://$(find unitree_go2_description)/meshes/calf.dae" scale="1 1 1"/>
+                    <!-- <mesh filename="file://$(find unitree_go2_description)/meshes/calf.dae" scale="1 1 1"/> -->
+                    <mesh filename="package://unitree_go2_description/meshes/link3.STL" />
                 </geometry>
             </visual>
@@ -135,7 +149,13 @@
         <link name="${name}_foot">
             <visual>
-                <origin rpy="0 0 0" xyz="0 0 0"/>
+                <xacro:if value="${mirror_dae == True}">
+                    <origin rpy="0 0 ${PI/2.0}" xyz="0 0 0"/>
+                </xacro:if>
+                <xacro:if value="${mirror_dae == False}">
+                    <origin rpy="0 0 ${-PI/2.0}" xyz="0 0 0"/>
+                </xacro:if>
                 <geometry>
                     <sphere radius="${foot_radius-0.01}"/>
+                    <!-- <mesh filename="package://unitree_go2_description/meshes/wheel_Link.STL" /> -->
                 </geometry>
             </visual>
@@ -143,5 +163,6 @@
                 <origin rpy="0 0 0" xyz="0 0 0"/>
                 <geometry>
-                    <sphere radius="${foot_radius}"/>
+                    <!-- <mesh filename="package://unitree_go2_description/meshes/wheel_Link.STL" /> -->
+                    <sphere radius="${foot_radius-0.01}"/>
                 </geometry>
             </collision>

File: legacy/unitree_go2_description/xacro/robot.xacro (robot description, xacro)
@@ -11,5 +11,6 @@
     <xacro:include filename="$(find unitree_go2_description)/xacro/leg.xacro"/>
     <xacro:include filename="$(find unitree_go2_description)/xacro/ros2_control.xacro"/>
-    <xacro:include filename="$(find unitree_go2_description)/xacro/gazebo.xacro"/>
+    <!-- 开启gazebo仿真 -->
+    <!-- <xacro:include filename="$(find unitree_go2_description)/xacro/gazebo.xacro"/> -->
     <!-- <xacro:stairs stairs="15" xpos="0" ypos="0" zpos="0" /> -->
     <!-- Rotor related joint and link is only for demonstrate location. -->
@@ -36,8 +37,9 @@
         <child link="trunk"/>
     </joint>
-    <xacro:include filename="$(find velodyne_description)/urdf/VLP-16.urdf.xacro"/>
+    <!-- gazebo专用 -->
+    <!-- <xacro:include filename="$(find velodyne_description)/urdf/VLP-16.urdf.xacro"/>
     <xacro:VLP-16 parent="trunk" name="rslidar" topic="/rslidar_points" organize_cloud="${organize_cloud}" hz="10" samples="440" gpu="${gpu}">
       <origin xyz="0.2 0 0.08" rpy="0 0 0" />
-    </xacro:VLP-16>
+    </xacro:VLP-16> -->
     <link name="camera_link">
     </link>
@@ -54,14 +56,14 @@
     <child link="camera_link_fake"/>
   </joint>
-<!-- <xacro:include filename="$(find realsense_ros2_gazebo)/xacro/depthcam.xacro"/>
-<xacro:realsense_R200 sensor_name="camera" parent_link="trunk" rate="30.0">
-  <origin rpy="0 0 0" xyz="0 0 0.5"/>
-</xacro:realsense_R200>
-  -->
+    <!-- <xacro:include filename="$(find realsense_ros2_gazebo)/xacro/depthcam.xacro"/>
+    <xacro:realsense_R200 sensor_name="camera" parent_link="trunk" rate="30.0">
+    <origin rpy="0 0 0" xyz="0 0 0.5"/>
+    </xacro:realsense_R200> -->
     <link name="trunk">
         <visual>
             <origin rpy="0 0 0" xyz="0 0 0"/>
             <geometry>
-                <mesh filename="file://$(find unitree_go2_description)/meshes/trunk.dae" scale="1 1 1"/>
+                <!-- <mesh filename="file://$(find unitree_go2_description)/meshes/trunk.dae" scale="1 1 1"/> -->
+                <box size="${trunk_length} ${trunk_width} ${trunk_height}"/>
             </geometry>
             <material name="orange"/>

File: legacy/unitree_go2_description/xacro/ros2_control.xacro (robot description, xacro)
@@ -1,5 +1,5 @@
 <?xml version="1.0"?>
 <robot xmlns:xacro="http://www.ros.org/wiki/xacro">
-    <xacro:arg name="IS_USING_GAZEBO" default="true"/>
+    <xacro:arg name="IS_USING_GAZEBO" default="false"/>
     <xacro:macro name="joint_interface" params="name">
         <joint name="${name}">
@@ -49,5 +49,13 @@
             <state_interface name="linear_acceleration.z"/>
         </sensor>
-        <sensor name="fl_ft_sensor">
+        <sensor name="foot_force">
+          <state_interface name="FL" />
+          <state_interface name="RL" />
+          <state_interface name="FR" />
+          <state_interface name="RR" />
+          <!-- <state_interface name="torque.y" />
+          <state_interface name="torque.z" /> -->
+        </sensor>
+        <!-- <sensor name="fl_ft_sensor">
           <state_interface name="force.x" />
           <state_interface name="force.y" />
@@ -108,5 +116,5 @@
           <param name="ty_range">15</param>
           <param name="tz_range">15</param>
-        </sensor>
+        </sensor> -->
     </ros2_control>
 </robot>
